Commit message: Addition of the "dog" model

File: assignment2/urdf/robot.xacro (robot description, xacro)
@@ -84,5 +84,5 @@
       <origin rpy="0 1.5707 1.5707" xyz="0 0 0"/>
       <xacro:wheel_geometry />
-      <material name="red"/>
+      <material name="orange"/>
     </visual>
   </link>
@@ -96,9 +96,86 @@
       <origin rpy="0 1.5707 1.5707" xyz="0 0 0"/>
       <xacro:wheel_geometry />
-      <material name="red"/>
-    </visual>
-  </link>
+      <material name="orange"/>
+    </visual>
+  </link>
+  <link name="link_neck">
+    <xacro:default_inertial mass="0.2"/>
+    <collision name="link_neck_collision">
+      <origin rpy="1.5707 1.5707 0" xyz="0 0.05 0"/>
+      <geometry>
+        <cylinder length="0.1" radius="0.04"/>
+      </geometry>
+    </collision>
+    <visual name="link_neck_visual">
+      <origin rpy="1.5707 1.5707 0" xyz="0 0.05 0"/>
+      <geometry>
+        <cylinder length="0.1" radius="0.04"/>
+      </geometry>
+      <material name="white"/>
+    </visual>
+  </link>
+  <link name="link_head">
+    <xacro:default_inertial mass="0.2"/>
+	    <collision>
+	      <origin xyz="0 0 0" rpy="0 0 0"/>
+	      <geometry>
+		      <box size="0.1 0.1 0.2"/>
+	      </geometry>
+	    </collision>
+	    <visual>
+	      <origin xyz="0 0 0" rpy="0 0 0"/>
+	      <geometry>
+		      <box size="0.1 0.1 0.2"/>
+	      </geometry>
+	      <material name="orange">
+	      </material>
+	    </visual>
+  </link>
+  <link name="camera_link">
+	    <collision>
+	      <origin xyz="0 0 0" rpy="0 0 0"/>
+	      <geometry>
+		<box size="0.05 0.05 0.05"/>
+	      </geometry>
+	    </collision>
+	    <visual>
+	      <origin xyz="0 0 0" rpy="0 0 0"/>
+	      <geometry>
+		<box size="0.05 0.05 0.05"/>
+	      </geometry>
+	      <material name="white">
+	      </material>
+	    </visual>
+	    <inertial>
+	      <mass value="1e-5" />
+	      <origin xyz="0 0 0" rpy="0 0 0"/>
+	      <inertia ixx="1e-6" ixy="0" ixz="0" iyy="1e-6" iyz="0" izz="1e-6" />
+	    </inertial>
+  </link>
+  <!--<link name="link_mouth">
+    <xacro:default_inertial mass="0.2"/>
+    <collision name="link_mouth_collision">
+      <origin rpy="0 0 0" xyz="0 0 0"/>
+      <geometry>
+        <box size="0.01 0.03 0.01"/>
+      </geometry>
+    </collision>
+    <visual name="link_mouth_visual">
+      <origin rpy="0 0 0" xyz="0 0 0"/>
+      <geometry>
+        <box size="0.01 0.03 0.01"/>
+      </geometry>
+      <material name="blue"/>
+    </visual>
+  </link>-->
+  <joint name="joint_neck" type="fixed">
+    <origin rpy="1.5707 0 0" xyz="0 0 0.035"/>
+    <child link="link_neck"/>
+    <parent link="link_chassis"/>
+    <!-- <axis rpy="0 0 0" xyz="0 1 0"/> -->
+    <axis rpy="0 0 0" xyz="0 0 0"/>
+  </joint>
   <joint name="joint_right_wheel" type="continuous">
-    <origin rpy="0 0 0" xyz="-0.05 0.15 0"/>
+    <origin rpy="0 0 0" xyz="-0.05 0.17 0"/>
     <child link="link_right_wheel"/>
     <parent link="link_chassis"/>
@@ -108,5 +185,5 @@
   </joint>
   <joint name="joint_left_wheel" type="continuous">
-    <origin rpy="0 0 0" xyz="-0.05 -0.15 0"/>
+    <origin rpy="0 0 0" xyz="-0.05 -0.17 0"/>
     <child link="link_left_wheel"/>
     <parent link="link_chassis"/>
@@ -115,31 +192,27 @@
     <joint_properties damping="1.0" friction="1.0"/>
   </joint>
-  <link name="camera_link">
-	    <collision>
-	      <origin xyz="0 0 0.025" rpy="0 0 0"/>
-	      <geometry>
-		<box size="0.05 0.05 0.05"/>
-	      </geometry>
-	    </collision>
-	    <visual>
-	      <origin xyz="0 0 0.025" rpy="0 0 0"/>
-	      <geometry>
-		<box size="0.05 0.05 0.05"/>
-	      </geometry>
-	      <material name="red">
-		<color rgba="1 0 0 1"/>
-	      </material>
-	    </visual>
-	    <inertial>
-	      <mass value="1e-5" />
-	      <origin xyz="0 0 0" rpy="0 0 0"/>
-	      <inertia ixx="1e-6" ixy="0" ixz="0" iyy="1e-6" iyz="0" izz="1e-6" />
-	    </inertial>
-  </link>
-  <joint name="camera_joint" type="fixed">
-	    <axis xyz="0 1 0" />
-	    <origin xyz="0.23 0 0.0" rpy="0 0 0"/>
-	    <parent link="link_chassis"/>
+  <joint name="head_joint" type="continuous">
+      <axis xyz="0 1 0"/>
+	    <origin xyz="0 0.15 0" rpy="0 0 0"/>
+	    <parent link="link_neck"/>
+	    <child link="link_head"/>
+      <!-- <limit effort="10000" lower="-1.8" upper="1.8" velocity="1000"/> -->
+      <limit effort="10000" velocity="1000"/>
+      <joint_properties damping="1.0" friction="1.0"/>
+	 </joint>
+    <joint name="camera_joint" type="fixed">
+      <axis xyz="0 0 1"/>
+      <!-- <axis xyz="0 0 1"/> -->
+	    <origin xyz="0.05 0 0" rpy="0 0 0"/>
+	    <parent link="link_head"/>
 	    <child link="camera_link"/>
 	 </joint>
+  <!--<joint name="joint_mouth" type="continuous">
+    <origin rpy="0 0 0" xyz="0 0.05 0"/>
+    <child link="camera_link"/>
+    <parent link="link_mouth"/>
+    <axis rpy="0 0 0" xyz="0 1 0"/>
+    <limit effort="10000" velocity="1000"/>
+    <joint_properties damping="1.0" friction="1.0"/>
+  </joint>-->
 </robot>

Commit message: Ball moving, normal & sleep working
Many file updates, but I starting to fear I will not be able to finish in time...

File: assignment2/urdf/robot.xacro (robot description, xacro)
@@ -40,5 +40,5 @@
     <color rgba="1.0 1.0 1.0 1.0"/>
   </material>
-	  <link name="link_chassis">
+	<link name="link_chassis">
     <!-- pose and inertial -->
     <pose>0 0 0.1 0 0 0</pose>
@@ -153,20 +153,4 @@
 	    </inertial>
   </link>
-  <!--<link name="link_mouth">
-    <xacro:default_inertial mass="0.2"/>
-    <collision name="link_mouth_collision">
-      <origin rpy="0 0 0" xyz="0 0 0"/>
-      <geometry>
-        <box size="0.01 0.03 0.01"/>
-      </geometry>
-    </collision>
-    <visual name="link_mouth_visual">
-      <origin rpy="0 0 0" xyz="0 0 0"/>
-      <geometry>
-        <box size="0.01 0.03 0.01"/>
-      </geometry>
-      <material name="blue"/>
-    </visual>
-  </link>-->
   <joint name="joint_neck" type="fixed">
     <origin rpy="1.5707 0 0" xyz="0 0 0.035"/>
@@ -192,14 +176,13 @@
     <joint_properties damping="1.0" friction="1.0"/>
   </joint>
-  <joint name="head_joint" type="continuous">
+  <joint name="head_joint" type="revolute">
       <axis xyz="0 1 0"/>
 	    <origin xyz="0 0.15 0" rpy="0 0 0"/>
 	    <parent link="link_neck"/>
 	    <child link="link_head"/>
-      <!-- <limit effort="10000" lower="-1.8" upper="1.8" velocity="1000"/> -->
-      <limit effort="10000" velocity="1000"/>
+      <limit effort="10000" lower="0.7854" upper="0.7854" velocity="1000"/>
       <joint_properties damping="1.0" friction="1.0"/>
 	 </joint>
-    <joint name="camera_joint" type="fixed">
+  <joint name="camera_joint" type="fixed">
       <axis xyz="0 0 1"/>
       <!-- <axis xyz="0 0 1"/> -->
@@ -207,12 +190,14 @@
 	    <parent link="link_head"/>
 	    <child link="camera_link"/>
-	 </joint>
-  <!--<joint name="joint_mouth" type="continuous">
-    <origin rpy="0 0 0" xyz="0 0.05 0"/>
-    <child link="camera_link"/>
-    <parent link="link_mouth"/>
-    <axis rpy="0 0 0" xyz="0 1 0"/>
-    <limit effort="10000" velocity="1000"/>
-    <joint_properties damping="1.0" friction="1.0"/>
-  </joint>-->
+	</joint>
+  <transmission name="head_joint_trans">
+	  <type>transmission_interface/SimpleTransmission</type>
+	  <joint name="head_joint">
+		  <hardwareInterface>hardware_interface/EffortJointInterface</hardwareInterface>
+	  </joint>
+	  <actuator name="motor1">
+		  <hardwareInterface>hardware_interface/EffortJointInterface</hardwareInterface>
+		  <mechanicalInterface>1</mechanicalInterface>
+	  </actuator>
+  </transmission>
 </robot>

Commit message: Many improvements (still to be tested)
code comments added, unnecessary stuff deleted

File: assignment2/urdf/robot.xacro (robot description, xacro)
@@ -177,9 +177,9 @@
   </joint>
   <joint name="head_joint" type="revolute">
-      <axis xyz="0 1 0"/>
+      <axis xyz="0 0 1"/> <!--<axis xyz="0 1 0"/>-->
 	    <origin xyz="0 0.15 0" rpy="0 0 0"/>
 	    <parent link="link_neck"/>
 	    <child link="link_head"/>
-      <limit effort="10000" lower="0.7854" upper="0.7854" velocity="1000"/>
+      <limit effort="10000" lower="-0.7854" upper="0.7854" velocity="1000"/>
       <joint_properties damping="1.0" friction="1.0"/>
 	 </joint>

Commit message: first working commit
now i just miss some readme stuff

File: assignment2/urdf/robot.xacro (robot description, xacro)
@@ -157,5 +157,4 @@
     <child link="link_neck"/>
     <parent link="link_chassis"/>
-    <!-- <axis rpy="0 0 0" xyz="0 1 0"/> -->
     <axis rpy="0 0 0" xyz="0 0 0"/>
   </joint>
@@ -177,5 +176,5 @@
   </joint>
   <joint name="head_joint" type="revolute">
-      <axis xyz="0 0 1"/> <!--<axis xyz="0 1 0"/>-->
+      <axis xyz="0 1 0"/>
 	    <origin xyz="0 0.15 0" rpy="0 0 0"/>
 	    <parent link="link_neck"/>
@@ -186,5 +185,4 @@
   <joint name="camera_joint" type="fixed">
       <axis xyz="0 0 1"/>
-      <!-- <axis xyz="0 0 1"/> -->
 	    <origin xyz="0.05 0 0" rpy="0 0 0"/>
 	    <parent link="link_head"/>
