Commit message: Made the eyes of the robot. still unsure about laser working or not
It does not appear in RViz but maybe I have to subscribe to topics?

File: assignment3/urdf/robot.xacro (robot description, xacro)
@@ -1,5 +1,5 @@
 <?xml version="1.0"?>
 <robot xmlns:xacro="http://www.ros.org/wiki/xacro" name="robot_xacro">
-<xacro:include filename="$(find assignment2)/urdf/robot.gazebo"/>
+<xacro:include filename="$(find assignment3)/urdf/robot.gazebo"/>
 	<xacro:property name="length_wheel" value="0.04" />
 	<xacro:property name="radius_wheel" value="0.1" />
@@ -144,5 +144,5 @@
 		<box size="0.03 0.03 0.03"/>
 	      </geometry>
-	      <material name="white">
+	      <material name="blue">
 	      </material>
 	    </visual>
@@ -165,5 +165,5 @@
 		<box size="0.03 0.03 0.03"/>
 	      </geometry>
-	      <material name="white">
+	      <material name="blue">
 	      </material>
 	    </visual>
@@ -206,12 +206,14 @@
 	</joint>
   <joint name="camera_joint" type="fixed">
-      <axis xyz="0 0 1"/>
-	    <origin xyz="0.05 -0.02 0" rpy="0 0 0"/>
+      <axis xyz="0 1 0"/> <!--<axis xyz="0 0 1"/>-->
+	    <!--<origin xyz="0.05 -0.02 0" rpy="0 0 0"/>-->
+      <origin xyz="0.05 0 -0.02" rpy="0 0 0"/> <!-- left eye of the robot -->
 	    <parent link="link_head"/>
 	    <child link="camera_link"/>
 	</joint>
   <joint name="laser_joint" type="fixed">
-      <axis xyz="0 0 1"/>
-	    <origin xyz="0.05 0.02 0" rpy="0 0 0"/>
+      <axis xyz="0 1 0"/> <!--<axis xyz="0 0 1"/>-->
+	    <!--<origin xyz="0.05 0.02 0" rpy="0 0 0"/>-->
+      <origin xyz="0.05 0 0.02" rpy="0 0 0"/> <!-- right eye of the robot -->
 	    <parent link="link_head"/>
 	    <child link="laser_link"/>

Commit message: Laser and map RViz problems solved, small adjustments, empty eye added

File: assignment3/urdf/robot.xacro (robot description, xacro)
@@ -69,5 +69,5 @@
     </collision>
     <visual name="caster_front_visual">
-      <origin rpy=" 0 0 0" xyz="0.2 0 -0.05"/>
+      <origin rpy="0 0 0" xyz="0.2 0 -0.05"/>
       <geometry>
         <sphere radius="0.05"/>
@@ -154,4 +154,25 @@
   </link>
   <link name="laser_link">
+	    <collision>
+	      <origin xyz="0 0 0" rpy="0 0 0"/>
+	      <geometry>
+		<box size="0.03 0.03 0.03"/>
+	      </geometry>
+	    </collision>
+	    <visual>
+	      <origin xyz="0 0 0" rpy="0 0 0"/>
+	      <geometry>
+		<box size="0.03 0.03 0.03"/>
+	      </geometry>
+	      <material name="orange">
+	      </material>
+	    </visual>
+	    <inertial>
+	      <mass value="1e-5" />
+	      <origin xyz="0 0 0" rpy="0 0 0"/>
+	      <inertia ixx="1e-6" ixy="0" ixz="0" iyy="1e-6" iyz="0" izz="1e-6" />
+	    </inertial>
+  </link>
+  <link name="link_eye">
 	    <collision>
 	      <origin xyz="0 0 0" rpy="0 0 0"/>
@@ -207,14 +228,18 @@
   <joint name="camera_joint" type="fixed">
       <axis xyz="0 1 0"/> <!--<axis xyz="0 0 1"/>-->
-	    <!--<origin xyz="0.05 -0.02 0" rpy="0 0 0"/>-->
-      <origin xyz="0.05 0 -0.02" rpy="0 0 0"/> <!-- left eye of the robot -->
+      <origin xyz="0.05 0 -0.02" rpy="0 0 0"/> <!-- left eye of the robot (camera) -->
 	    <parent link="link_head"/>
 	    <child link="camera_link"/>
 	</joint>
+  <joint name="eye_joint" type="fixed">
+      <axis xyz="0 1 0"/> <!--<axis xyz="0 0 1"/>-->
+      <origin xyz="0.05 0 0.02" rpy="0 0 0"/> <!-- right eye of the robot (empty) -->
+	    <parent link="link_head"/>
+	    <child link="link_eye"/>
+	</joint>
   <joint name="laser_joint" type="fixed">
       <axis xyz="0 1 0"/> <!--<axis xyz="0 0 1"/>-->
-	    <!--<origin xyz="0.05 0.02 0" rpy="0 0 0"/>-->
-      <origin xyz="0.05 0 0.02" rpy="0 0 0"/> <!-- right eye of the robot -->
-	    <parent link="link_head"/>
+      <origin xyz="0.254 0 0.03" rpy="0 0 0"/>
+	    <parent link="link_chassis"/>
 	    <child link="laser_link"/>
 	</joint>

Commit message: First relatively big debugging session completed
Still need to test the first_run of explore.cpp, and to solve the sprouting laser problem

File: assignment3/urdf/robot.xacro (robot description, xacro)
@@ -8,5 +8,6 @@
                        <mass value="${mass}" />
                        <origin rpy="0 1.5707 1.5707" xyz="0 0 0"/>
-                       <inertia ixx="0.000526666666667" ixy="0" ixz="0" iyy="0.000526666666667" iyz="0" izz="0.001"/>
+                       <inertia ixx="0.000526666666667" ixy="0" ixz="0"
+                                iyy="0.000526666666667" iyz="0" izz="0.001"/>
                </inertial>
 	</xacro:macro>
@@ -46,5 +47,6 @@
       <mass value="5"/>
       <origin rpy="0 0 0" xyz="0 0 0.1"/>
-      <inertia ixx="0.0395416666667" ixy="0" ixz="0" iyy="0.106208333333" iyz="0" izz="0.106208333333"/>
+      <inertia ixx="0.0395416666667" ixy="0" ixz="0" iyy="0.106208333333"
+                                     iyz="0" izz="0.106208333333"/>
     </inertial>
     <!-- body -->
@@ -63,5 +65,5 @@
     <!-- caster front -->
     <collision name="caster_front_collision">
-      <origin rpy=" 0 0 0" xyz="0.35 0 -0.05"/>
+      <origin rpy="0 0 0" xyz="0.35 0 -0.05"/>
       <geometry>
         <sphere radius="0.05"/>
@@ -217,5 +219,4 @@
     <joint_properties damping="1.0" friction="1.0"/>
   </joint>
-  <!--<joint name="head_joint" type="revolute">-->
   <joint name="head_joint" type="fixed">
       <axis xyz="0 1 0"/>
@@ -223,6 +224,4 @@
 	    <parent link="link_neck"/>
 	    <child link="link_head"/>
-      <!--<limit effort="10000" lower="-0.7854" upper="0.7854" velocity="1000"/>-->
-      <!--<joint_properties damping="1.0" friction="1.0"/>-->
 	</joint>
   <joint name="camera_joint" type="fixed">
@@ -244,13 +243,3 @@
 	    <child link="laser_link"/>
 	</joint>
-  <!--<transmission name="head_joint_trans">
-	  <type>transmission_interface/SimpleTransmission</type>
-	  <joint name="head_joint">
-		  <hardwareInterface>hardware_interface/EffortJointInterface</hardwareInterface>
-	  </joint>
-	  <actuator name="motor1">
-		  <hardwareInterface>hardware_interface/EffortJointInterface</hardwareInterface>
-		  <mechanicalInterface>1</mechanicalInterface>
-	  </actuator>
-  </transmission>-->
 </robot>

Commit message: Fixed robot model; still working on first_run for explore.cpp

File: assignment3/urdf/robot.xacro (robot description, xacro)
@@ -53,5 +53,5 @@
     <collision name="collision_chassis">
       <geometry>
-        <box size="0.5 0.3 0.07"/>
+        <box size="0.45 0.3 0.07"/>
       </geometry>
     </collision>
@@ -59,5 +59,5 @@
       <origin rpy="0 0 0" xyz="0 0 0"/>
       <geometry>
-        <box size="0.5 0.3 0.07"/>
+        <box size="0.45 0.3 0.07"/>
       </geometry>
       <material name="blue"/>
@@ -65,5 +65,5 @@
     <!-- caster front -->
     <collision name="caster_front_collision">
-      <origin rpy="0 0 0" xyz="0.35 0 -0.05"/>
+      <origin rpy="0 0 0" xyz="0.15 0 -0.05"/>
       <geometry>
         <sphere radius="0.05"/>
@@ -71,5 +71,5 @@
     </collision>
     <visual name="caster_front_visual">
-      <origin rpy="0 0 0" xyz="0.2 0 -0.05"/>
+      <origin rpy="0 0 0" xyz="0.15 0 -0.05"/>
       <geometry>
         <sphere radius="0.05"/>
@@ -150,7 +150,7 @@
 	    </visual>
 	    <inertial>
-	      <mass value="1e-5" />
-	      <origin xyz="0 0 0" rpy="0 0 0"/>
-	      <inertia ixx="1e-6" ixy="0" ixz="0" iyy="1e-6" iyz="0" izz="1e-6" />
+	      <mass value="1e-5"/>
+	      <origin xyz="0 0 0" rpy="0 0 0"/>
+	      <inertia ixx="1e-6" ixy="0" ixz="0" iyy="1e-6" iyz="0" izz="1e-6"/>
 	    </inertial>
   </link>
@@ -171,7 +171,7 @@
 	    </visual>
 	    <inertial>
-	      <mass value="1e-5" />
-	      <origin xyz="0 0 0" rpy="0 0 0"/>
-	      <inertia ixx="1e-6" ixy="0" ixz="0" iyy="1e-6" iyz="0" izz="1e-6" />
+	      <mass value="1e-5"/>
+	      <origin xyz="0 0 0" rpy="0 0 0"/>
+	      <inertia ixx="1e-6" ixy="0" ixz="0" iyy="1e-6" iyz="0" izz="1e-6"/>
 	    </inertial>
   </link>
@@ -192,7 +192,7 @@
 	    </visual>
 	    <inertial>
-	      <mass value="1e-5" />
-	      <origin xyz="0 0 0" rpy="0 0 0"/>
-	      <inertia ixx="1e-6" ixy="0" ixz="0" iyy="1e-6" iyz="0" izz="1e-6" />
+	      <mass value="1e-5"/>
+	      <origin xyz="0 0 0" rpy="0 0 0"/>
+	      <inertia ixx="1e-6" ixy="0" ixz="0" iyy="1e-6" iyz="0" izz="1e-6"/>
 	    </inertial>
   </link>
@@ -239,5 +239,5 @@
   <joint name="laser_joint" type="fixed">
       <axis xyz="0 1 0"/> <!--<axis xyz="0 0 1"/>-->
-      <origin xyz="0.254 0 0.03" rpy="0 0 0"/>
+      <origin xyz="0.212 0 0.021" rpy="0 0 0"/>
 	    <parent link="link_chassis"/>
 	    <child link="laser_link"/>

Commit message: Many improvements & corrections, but the robot is still heavily jerking
Tried to solve by changing parameters of gmapping, base_local_planner,  move_base, xacro cmd_vel rate and robot torque, and by disabling various nodes one at a time. Still no luck. The problem is probably related to this one: https://answers.ros.org/question/339017/move_base-how-to-move-robot-smoothly/

File: assignment3/urdf/robot.xacro (robot description, xacro)
@@ -226,17 +226,17 @@
 	</joint>
   <joint name="camera_joint" type="fixed">
-      <axis xyz="0 1 0"/> <!--<axis xyz="0 0 1"/>-->
-      <origin xyz="0.05 0 -0.02" rpy="0 0 0"/> <!-- left eye of the robot (camera) -->
+      <axis xyz="0 1 0"/>
+      <origin xyz="0.05 0 -0.02" rpy="-1.5707 0 0"/> <!-- left eye of the robot (camera) -->
 	    <parent link="link_head"/>
 	    <child link="camera_link"/>
 	</joint>
   <joint name="eye_joint" type="fixed">
-      <axis xyz="0 1 0"/> <!--<axis xyz="0 0 1"/>-->
-      <origin xyz="0.05 0 0.02" rpy="0 0 0"/> <!-- right eye of the robot (empty) -->
+      <axis xyz="0 1 0"/>
+      <origin xyz="0.05 0 0.02" rpy="-1.5707 0 0"/> <!-- right eye of the robot (empty) -->
 	    <parent link="link_head"/>
 	    <child link="link_eye"/>
 	</joint>
   <joint name="laser_joint" type="fixed">
-      <axis xyz="0 1 0"/> <!--<axis xyz="0 0 1"/>-->
+      <axis xyz="0 1 0"/>
       <origin xyz="0.212 0 0.021" rpy="0 0 0"/>
 	    <parent link="link_chassis"/>

Commit message: Finally solved the jerking robot issue
It was a problem with the caster. Note to future self: if it ain't broke, don't fix it!

File: assignment3/urdf/robot.xacro (robot description, xacro)
@@ -47,6 +47,6 @@
       <mass value="5"/>
       <origin rpy="0 0 0" xyz="0 0 0.1"/>
-      <inertia ixx="0.0395416666667" ixy="0" ixz="0" iyy="0.106208333333"
-                                     iyz="0" izz="0.106208333333"/>
+      <inertia ixx="0.0395416666667" ixy="0" ixz="0"
+               iyy="0.106208333333" iyz="0" izz="0.106208333333"/>
     </inertial>
     <!-- body -->
@@ -65,5 +65,5 @@
     <!-- caster front -->
     <collision name="caster_front_collision">
-      <origin rpy="0 0 0" xyz="0.15 0 -0.05"/>
+      <origin rpy="0 0 0" xyz="0.35 0 -0.05"/>
       <geometry>
         <sphere radius="0.05"/>

Commit message: Major update (see description)
Readme & doxygen corrections, gmapping bug (hopefully) mostly sovled, launch files reorganized and cleaned, rviz config redone, xacro and gazebo dog models corrected, many yaml parametes reset to default or corrected, "house2.world" renamed to "house.world"

File: assignment3/urdf/robot.xacro (robot description, xacro)
@@ -102,5 +102,5 @@
   </link>
   <link name="link_neck">
-    <xacro:default_inertial mass="0.2"/>
+    <xacro:default_inertial mass="0.02"/>
     <collision name="link_neck_collision">
       <origin rpy="1.5707 1.5707 0" xyz="0 0.05 0"/>
@@ -118,5 +118,5 @@
   </link>
   <link name="link_head">
-    <xacro:default_inertial mass="0.2"/>
+    <xacro:default_inertial mass="0.02"/>
 	    <collision>
 	      <origin xyz="0 0 0" rpy="0 0 0"/>
@@ -201,5 +201,4 @@
     <child link="link_neck"/>
     <parent link="link_chassis"/>
-    <axis rpy="0 0 0" xyz="0 0 0"/>
   </joint>
   <joint name="joint_right_wheel" type="continuous">
@@ -220,5 +219,4 @@
   </joint>
   <joint name="head_joint" type="fixed">
-      <axis xyz="0 1 0"/>
 	    <origin xyz="0 0.15 0" rpy="0 0 0"/>
 	    <parent link="link_neck"/>
@@ -226,5 +224,4 @@
 	</joint>
   <joint name="camera_joint" type="fixed">
-      <axis xyz="0 1 0"/>
       <origin xyz="0.05 0 -0.02" rpy="-1.5707 0 0"/> <!-- left eye of the robot (camera) -->
 	    <parent link="link_head"/>
@@ -232,5 +229,4 @@
 	</joint>
   <joint name="eye_joint" type="fixed">
-      <axis xyz="0 1 0"/>
       <origin xyz="0.05 0 0.02" rpy="-1.5707 0 0"/> <!-- right eye of the robot (empty) -->
 	    <parent link="link_head"/>
@@ -238,6 +234,5 @@
 	</joint>
   <joint name="laser_joint" type="fixed">
-      <axis xyz="0 1 0"/>
-      <origin xyz="0.212 0 0.021" rpy="0 0 0"/>
+      <origin xyz="0.226 0 0.036" rpy="0 0 0"/>
 	    <parent link="link_chassis"/>
 	    <child link="laser_link"/>
